File: hardware/RS232TTL_Adaper/RS232TTL_Adaper.kicad_pcb (KiCad board)
At the start: 2 copper layers, 58.4 x 54 mm, 8 parts, among them J1 DB25_Male, J2 Conn_01x05, U1 MAX232N

Commit message: moved graphics
Parts:
- added REF**: OSHW-Logo2_9.8x8mm_SilkScreen, Symbol:OSHW-Logo2_9.8x8mm_SilkScreen, F.Cu at (110.4, 92.8)
Other:
- board text added: "Master Control Board R232 to TTL Adapter v1.0"

Commit message: remove connection to +/- 12v
Parts:
- removed REF**: OSHW-Logo2_9.8x8mm_SilkScreen, Symbol:OSHW-Logo2_9.8x8mm_SilkScreen
Connections:
- C3 pad 1: /VS+ -> Net-(U1-Pad2)
- C3 pad 2: GND -> +5V
- C4 pad 1: +5V -> GND
- C4 pad 2: /VS- -> Net-(U1-Pad6)
- J1 pad 12: /VS+ -> unconnected-(J1-Pad12)
- J1 pad 25: /VS- -> unconnected-(J1-Pad25)
- U1 pad 2: /VS+ -> Net-(U1-Pad2)
- U1 pad 6: /VS- -> Net-(U1-Pad6)
Routing:
- net +5V: track 61.7 -> 0.00 mm
- net /VS-: track 48.0 -> 0.00 mm
- net /VS+: track 24.3 -> 0.00 mm
- net Net-(U1-Pad6): track 0.00 -> 9.78 mm
- net Net-(U1-Pad2): track 0.00 -> 9.31 mm
- net /RX_232: track 29.6 -> 24.8 mm
- net /TX_232: track 31.0 -> 29.3 mm
- added copper zone on F.Cu, net +5V
