File: hardware/SerialClockFlyover/SerialClockFlyover.kicad_sch (KiCad schematic)
At the start: 0 parts

Commit message: added 15M resistor
Parts:
- added J1: Conn_02x13_Odd_Even, Connector_PinSocket_2.54mm:PinSocket_2x13_P2.54mm_Vertical, symbol Connector_Generic:Conn_02x13_Odd_Even
- added J2: Conn_02x09_Odd_Even, Connector_PinHeader_2.54mm:PinHeader_2x09_P2.54mm_Vertical, symbol Connector_Generic:Conn_02x09_Odd_Even
- added J3: Conn_01x05, Connector_PinHeader_2.54mm:PinHeader_1x05_P2.54mm_Vertical, symbol Connector_Generic:Conn_01x05
- added R1, R2, R3: 1K, Resistor_THT:R_Axial_DIN0207_L6.3mm_D2.5mm_P10.16mm_Horizontal, symbol Device:R
- added R4: 15M, Resistor_THT:R_Axial_DIN0207_L6.3mm_D2.5mm_P10.16mm_Horizontal, symbol Device:R
- added S1: 1825910-6, digikey-footprints:Switch_Tactile_THT_6x6mm, symbol dk_Tactile-Switches:1825910-6
- added U1: MC14411P, Package_DIP:DIP-24_W15.24mm_Socket, symbol mcb:MC14411P
- added Y1: 1.8432 MHz, Crystal:Crystal_HC18-U_Vertical, symbol Device:Crystal_Small
Connections:
- new net: R4.1, U1.20 (XTALOUT), Y1.1
- new net: R4.2, U1.21 (XTALIN), Y1.2
- new net: J1.13 (Pin_13), J1.14 (Pin_14), J1.5 (Pin_5), J2.10 (Pin_10), J2.12 (Pin_12), J2.14 (Pin_14), J2.16 (Pin_16), J2.18 (Pin_18), J2.2 (Pin_2), J2.4 (Pin_4), J2.6 (Pin_6), J2.8 (Pin_8)
- new net: R2.2, U1.22 (RSB)
- new net: R1.2, U1.23 (RSA)
- new net: R3.2, S1.3, S1.4, U1.10 (~{RESET})
- new net +5V: J1.25 (Pin_25), R1.1, R2.1, R3.1, U1.24 (VDD)
- new net CTSB: J1.1 (Pin_1), J3.2 (Pin_2)
- new net F115200: J2.17 (Pin_17), U1.19 (F16)
- new net F1200: J2.3 (Pin_3), U1.7 (F9)
- new net F19200: J2.11 (Pin_11), U1.2 (F3)
- new net F2400: J2.5 (Pin_5), U1.5 (F8)
- new net F300: J2.1 (Pin_1), U1.9 (F14)
- new net F38400: J2.13 (Pin_13), U1.1 (F1)
- new net F4800: J2.7 (Pin_7), U1.4 (F7)
- new net F57600: J2.15 (Pin_15), U1.18 (F15)
- new net F9600: J2.9 (Pin_9), U1.3 (F5)
- new net GND: J1.26 (Pin_26), J3.1 (Pin_1), S1.1, S1.2, U1.12 (VSS)
- new net RTSB: J1.4 (Pin_4), J3.3 (Pin_3)
- new net RxDB: J1.7 (Pin_7), J3.5 (Pin_5)
- new net TxDB: J1.6 (Pin_6), J3.4 (Pin_4)
- no-connect marks 0 -> 24
