File: hardware/SerialClockFlyover/SerialClockFlyover.kicad_pcb (KiCad board)
At the start: 2 copper layers, 62.2 x 39.4 mm, 10 parts, among them J1 Conn_02x13_Odd_Even, J2 Conn_02x09_Odd_Even, J3 Conn_01x05, U1 MC14411P, Y1 1.8432 MHz

Commit message: added OSHW logo
Parts:
- added REF**: OSHW-Logo2_7.3x6mm_SilkScreen, Symbol:OSHW-Logo2_7.3x6mm_SilkScreen, F.Cu at (153.3, 87.0)
